Commit message: arm_with_tracer

File: social_system/robotic_arm/arm/rm_65_description/urdf/rm_65_flange.urdf.xacro (robot description, xacro)
@@ -423,4 +423,16 @@
     <parent link="Link6" />
     <child link="tool_link" />
+  </joint>
+<!-- camera  <mesh  filename="package://rm_65_description/meshes/akdk_camera_cad1.STL" />
+          <box size="0.2 0.3 0.3"/>
+          -->
+<!-- kinect -->
+  <xacro:include filename="$(find rm_65_description)/urdf/yixiuge_d435i.xacro" />
+  <!--添加d435i的link即joint -->
+  <xacro:yixiuge_d435i>     </xacro:yixiuge_d435i>
+  <joint name="yixiuge_kinect_base_joint" type="fixed">
+    <origin xyz="0.025 0.0 0.0" rpy="0 0 0" />
+    <parent link="tool_link"/>
+    <child link="camera_base_link"/>
   </joint>
     <!-- Transmissions for ROS Control -->

File: social_system/robotic_arm/arm/rm_65_description/urdf/rm_65_with_turtle.urdf.xacro (robot description, xacro)
@@ -1,14 +1,14 @@
 <?xml version="1.0" ?>
 <robot name="rm_65" xmlns:xacro="http://www.ros.org/wiki/xacro">
-<xacro:include filename="$(find rm_65_description)/urdf/rm_65.transmission.xacro"/>
-<xacro:include filename="$(find rm_65_description)/urdf/rm_65.gazebo.xacro"/>
-<!-- <xacro:include filename="$(find rm_65_description)/urdf/common.gazebo.xacro"/> -->
-<!-- Inertial matrix -->
-<xacro:macro name="inertial_matrix" params="mass">
-<inertial>
-    <mass value="${mass}" />
-    <inertia ixx="1.0" ixy="0.0" ixz="0.0" iyy="0.5" iyz="0.0" izz="1.0" />
-</inertial>
-</xacro:macro>
+  <xacro:include filename="$(find rm_65_description)/urdf/rm_65.transmission.xacro"/>
+  <xacro:include filename="$(find rm_65_description)/urdf/rm_65.gazebo.xacro"/>
+  <!-- <xacro:include filename="$(find rm_65_description)/urdf/common.gazebo.xacro"/> -->
+  <!-- Inertial matrix -->
+  <xacro:macro name="inertial_matrix" params="mass">
+    <inertial>
+        <mass value="${mass}" />
+        <inertia ixx="1.0" ixy="0.0" ixz="0.0" iyy="0.5" iyz="0.0" izz="1.0" />
+    </inertial>
+  </xacro:macro>
   <link
     name="turtle_link">
