Commit message: 7月3备份

File: social_system/robotic_arm/arm/rm_65_description/urdf/rm_65_with_d435i_with_tracer.urdf.xacro (robot description, xacro)
@@ -11,4 +11,5 @@
     </inertial>
   </xacro:macro>
+  <!-- below is tracer -->
   <xacro:arg name="robot_namespace" default="/" />
   <xacro:arg name="urdf_extras" default="empty.urdf" />
@@ -119,8 +120,13 @@
   </xacro:rl_wheel>
   <!-- Additional definitions -->
-  <xacro:include filename="$(arg urdf_extras)" />
+  <!-- <xacro:include filename="$(arg urdf_extras)" /> -->
   <!-- Gazebo definitions  -->
   <xacro:include filename="$(find tracer_description)/urdf/tracer.gazebo" />
-  <!-- 以下是机械臂 -->
+<joint name="tracer_joint" type="fixed">
+      <origin xyz="0 0 0.0" rpy="0 0 3.14" />
+      <parent link="tracer_link"/>
+      <child link="base_link"/>
+  </joint>
+  <!-- Below is arm robot -->
   <link
     name="base_link">

File: social_system/robotic_arm/arm/rm_65_description/urdf/rm_65_with_turtle.urdf.xacro (robot description, xacro)
@@ -454,5 +454,5 @@
       effort="300"
       velocity="1" />
-	<dynamics damping="50" friction="1"/>
+	  <dynamics damping="50" friction="1"/>
   </joint>
     <!-- Transmissions for ROS Control -->
